File: g473_generic_gen1_board.kicad_sch (KiCad schematic)
At the start: 40 parts

Commit message: a
Parts:
- removed J?: Conn_01x03_Pin, Connector_PinHeader_2.54mm:PinHeader_1x03_P2.54mm_Vertical, symbol Connector:Conn_01x03_Pin
- removed J?: Conn_01x09_Socket, Connector_PinSocket_2.54mm:PinSocket_1x09_P2.54mm_Vertical, symbol Connector:Conn_01x09_Socket
- removed J?: Conn_01x12_Socket, Connector_PinSocket_2.54mm:PinSocket_1x12_P2.54mm_Vertical, symbol Connector:Conn_01x12_Socket
- added C1: 1u, Capacitor_SMD:C_0603_1608Metric, symbol Device:C
- added C19, C21: 0.1u, Capacitor_SMD:C_0603_1608Metric, symbol Device:C
- added C3: 0.01u, Capacitor_SMD:C_0603_1608Metric, symbol Device:C
- added C4: 10u, Capacitor_SMD:C_0603_1608Metric, symbol Device:C
- added D5: UDZV5.1B, Diode_SMD:D_SOD-323, symbol Device:D_Zener
- added J4: Conn_02x10_Odd_Even, Connector_PinSocket_2.54mm:PinSocket_2x10_P2.54mm_Vertical, symbol Connector_Generic:Conn_02x10_Odd_Even
- added LS1: Speaker_Ultrasound, Buzzer_Beeper:Buzzer_Murata_PKLCS1212E, symbol Device:Speaker_Ultrasound
- added R7: 1k, Resistor_SMD:R_0603_1608Metric, symbol Device:R
- added SW3: SW_SPDT, My_Parts:SW_Slide_SPDT_Angled_SK-12D11VG3, symbol Switch:SW_SPDT
- added U1: TAR5SB33, Package_TO_SOT_SMD:SOT-23-5, symbol My_Parts:TAR5SB33
- added U5: TCK108AF, Package_TO_SOT_SMD:SOT-23-5, symbol My_Parts:TCK108AF
- D3, D4: renamed from D?; value D -> CUHS20S30
- J1, J5, J8: renamed from J?; footprint Connector_PinHeader_2.54mm:PinHeader_1x06_P2.54mm_Horizontal -> My_Parts:Neltron_3750R-06_1x06_P2.54mm_Horizontal
- J2, J7: renamed from J?; footprint Connector_PinHeader_2.54mm:PinHeader_1x04_P2.54mm_Horizontal -> My_Parts:Neltron_3750R-04_1x04_P2.54mm_Horizontal
- SW1, SW2: renamed from SW?; footprint Button_Switch_SMD:SW_Push_1P1T_NO_6x6mm_H9.5mm -> Button_Switch_THT:SW_PUSH_6mm
- gave numbers to parts that had none: 28
Connections:
- net +3V3: now also D1.2 (A), D2.2 (A), C4.1, J4.18 (Pin_18), U1.5 (OUT); no longer R1.1, R2.1
- net +5V: now also C1.1, C19.1, J4.19 (Pin_19), SW3.2 (B), U1.1 (IN), U1.3 (CTRL), U5.5 (IN)
- net +5V_ENC: now also C21.1, U5.1 (OUT)
- net ENC_EN: now also U3.38 (PA15), U5.3 (~{CTRL}); no longer U3.45 (PB7)
- net GND: now also C1.2, C19.2, C21.2, C3.2, C4.2, D5.2 (A), J4.20 (Pin_20), LS1.2, U1.2 (GND), U5.2 (GND)
- net LED_ERROR: now also R1.2; no longer D1.1 (K)
- net LED_STATUS: now also R2.2; no longer D2.1 (K)
- net PA0: now also J4.8 (Pin_8)
- net PA1: now also J4.9 (Pin_9)
- net PA10: now also J4.17 (Pin_17)
- net PA2: now also J4.10 (Pin_10)
- net PA3: now also J4.11 (Pin_11)
- net PA8: now also J4.15 (Pin_15)
- net PA9: now also J4.16 (Pin_16)
- net PB0: now also J4.12 (Pin_12)
- net PB1: now also J4.13 (Pin_13)
- net PB12: now also J4.14 (Pin_14)
- net PB3: now also J4.1 (Pin_1)
- net PB4: now also J4.2 (Pin_2)
- net PB5: now also J4.3 (Pin_3)
- net PB6: now also J4.4 (Pin_4)
- net PB8: now also J4.5 (Pin_5)
- net PB9: now also J4.6 (Pin_6)
- net PC13: now also J4.7 (Pin_7)
- net SW: now also U3.45 (PB7); no longer U3.38 (PA15)
- net UART4_RX: now also J1.5 (Pin_5)
- net UART4_TX: now also J1.6 (Pin_6)
- net at D3.2 (A), J1.2 (Pin_2): now also SW3.1 (A)
- net at D4.2 (A), J2.2 (Pin_2): now also SW3.3 (C)
- net PA4 renamed DAC1_OUT1
- net DAC1_OUT1: now also R7.2
- new net: D2.1 (K), R2.1
- new net: D1.1 (K), R1.1
- new net: D5.1 (K), LS1.1, R7.1
- new net: C3.1, U1.4 (NOISE)
Other:
- moved on the sheet: D1, D2, R1, R2
